File: Schematics/Main/PAM8403-Board.kicad_sch (KiCad schematic)
At the start: 1 part, among them U1 PAM8403D

Commit message: Added PAM8403-Board schematic
Parts:
- added C1, C15, C18, C19: 1 μF, symbol Device:C_Small
- added C16, C17: 10 μF, symbol Device:C_Small
- added C20, C21: 220 nF, symbol Device:C_Small
- added R1, R9: 10 kΩ, symbol Device:R
Connections:
- net GND: now also U1.11 (GND), U1.15 (PGND), U1.2 (PGND), C1.1, C15.2, C16.2, C17.2, C18.2, C19.1
- net LIN: now also C20.1
- net LOUT+: now also U1.1 (LOUT+)
- net LOUT-: now also U1.3 (LOUT-)
- net RIN: now also C21.1
- net ROUT+: now also U1.16 (ROUT+)
- net ROUT-: now also U1.14 (ROUT-)
- net at U1.10 (INR): now also R9.2
- net VDD: now reaches U1.12 (~{SHDN})
- net VDD: now also U1.13 (PVDD), U1.4 (PVDD), U1.5 (~{MUTE}), U1.6 (VDD), C1.2, C15.1, C16.1, C17.1, C18.1
- net at U1.7 (INL): now also R1.2
- net at U1.8 (VREF): now also C19.2
- new net: C20.2, R1.1
- new net: C21.2, R9.1
